File: pcb/pcb.kicad_sch (KiCad schematic)
At the start: 45 parts, among them J1 USB_C_Receptacle_USB2.0_14P, J10 SWDIO, J11 SWCLK, J12 USART1 TX, J13 USART1 RX, J14 GND, J15 3.3v, J16 GND, J17 NRST, J2 +3.3V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

Commit message: add pwr switch
Parts:
- added SW1: PWR SWITCH, Connector_PinSocket_2.54mm:PinSocket_1x02_P2.54mm_Vertical, symbol Switch:SW_DPST_x2
Connections:
- net +3.3V: now also SW1.2 (B); no longer C2.1, C8.1, L1.2, R1.1
- new net: C2.1, C8.1, L1.2, R1.1, SW1.1 (A)
Changed lines of the file:
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@@
 	)
 	(junction
-		(at 99.06 34.29)
+		(at 172.72 27.94)
 		(diameter 0)
 		(color 0 0 0 0)
 	)
 	(junction
-		(at 172.72 27.94)
+		(at 153.67 53.34)
 		(diameter 0)
 		(color 0 0 0 0)
 	)
 	(junction
-		(at 153.67 53.34)
+		(at 99.06 34.29)
 		(diameter 0)
 		(color 0 0 0 0)
@@
 	(wire
 		(pts
-			(xy 153.67 154.94) (xy 151.13 154.94)
-		)
-		(stroke
-			(width 0)
-			(type default)
-		)
-	)
-	(wire
-		(pts
 			(xy 133.35 74.93) (xy 127 74.93)
 		)
@@
 	(wire
 		(pts
-			(xy 153.67 160.02) (xy 153.67 154.94)
-		)
-		(stroke
-			(width 0)
-			(type default)
-		)
-	)
-	(wire
-		(pts
 			(xy 255.27 149.86) (xy 259.08 149.86)
 		)
@@
 	(wire
 		(pts
+			(xy 151.13 154.94) (xy 151.13 160.02)
+		)
+		(stroke
+			(width 0)
+			(type default)
+		)
+	)
+	(wire
+		(pts
 			(xy 72.39 93.98) (xy 78.74 93.98)
 		)
@@
 	(wire
 		(pts
+			(xy 151.13 154.94) (xy 153.67 154.94)
+		)
+		(stroke
+			(width 0)
+			(type default)
+		)
+	)
+	(wire
+		(pts
 			(xy 251.46 91.44) (xy 261.62 91.44)
 		)
@@
 	(symbol
 		(lib_id "power:+3.3V")
+		(at 151.13 160.02 180)
+		(unit 1)
+		(exclude_from_sim no)
+		(in_bom yes)
+		(on_board yes)
+		(dnp no)
+		(fields_autoplaced yes)
+		(property "Reference" "#PWR06"
+			(at 151.13 156.21 0)
+			(effects
+				(font
+					(size 1.27 1.27)
+				)
+				(hide yes)
+			)
+		)
+		(property "Value" "+3.3V"
+			(at 148.59 161.2901 0)
+			(effects
+				(font
+					(size 1.27 1.27)
+				)
+				(justify left)
+			)
+		)
+		(property "Footprint" ""
+			(at 151.13 160.02 0)
+			(effects
+				(font
+					(size 1.27 1.27)
+				)
+				(hide yes)
+			)
+		)
+		(property "Datasheet" ""
+			(at 151.13 160.02 0)
+			(effects
+				(font
+					(size 1.27 1.27)
+				)
+				(hide yes)
+			)
+		)
+		(property "Description" "Power symbol creates a global label with name \"+3.3V\""
+			(at 151.13 160.02 0)
+			(effects
+				(font
+					(size 1.27 1.27)
+				)
+				(hide yes)
+			)
+		)
+		(pin "1"
+		)
+		(instances
+			(project "pcb"
+				(path "/a02550bc-85b4-480d-868d-ccdfd0f6046d"
+					(reference "#PWR06")
+					(unit 1)
+				)
+			)
+		)
+	)
+	(symbol
+		(lib_id "power:+3.3V")
 		(at 179.07 77.47 270)
 		(unit 1)
@@
 	)
 	(symbol
-		(lib_id "power:+3.3V")
-		(at 153.67 160.02 180)
-		(unit 1)
-		(exclude_from_sim no)
-		(in_bom yes)
-		(on_board yes)
-		(dnp no)
-		(fields_autoplaced yes)
-		(property "Reference" "#PWR011"
-			(at 153.67 156.21 0)
-			(effects
-				(font
-					(size 1.27 1.27)
-				)
-				(hide yes)
-			)
-		)
-		(property "Value" "+3.3V"
-			(at 151.13 161.2901 0)
-			(effects
-				(font
-					(size 1.27 1.27)
-				)
-				(justify left)
-			)
-		)
-		(property "Footprint" ""
-			(at 153.67 160.02 0)
-			(effects
-				(font
-					(size 1.27 1.27)
-				)
-				(hide yes)
-			)
-		)
-		(property "Datasheet" ""
-			(at 153.67 160.02 0)
-			(effects
-				(font
-					(size 1.27 1.27)
-				)
-				(hide yes)
-			)
-		)
-		(property "Description" "Power symbol creates a global label with name \"+3.3V\""
-			(at 153.67 160.02 0)
-			(effects
-				(font
-					(size 1.27 1.27)
-				)
-				(hide yes)
-			)
-		)
-		(pin "1"
-		)
-		(instances
-			(project ""
-				(path "/a02550bc-85b4-480d-868d-ccdfd0f6046d"
-					(reference "#PWR011")
-					(unit 1)
-				)
-			)
-		)
-	)
-	(symbol
 		(lib_id "Device:C_Small")
 		(at 92.71 147.32 0)
@@
 	)
 	(symbol
-		(lib_id "Device:R_Small")
-		(at 260.35 35.56 90)
+		(lib_id "Switch:SW_DPST_x2")
+		(at 99.06 29.21 90)
 		(unit 1)
 		(exclude_from_sim no)
@@
 		(dnp no)
 		(fields_autoplaced yes)
-		(property "Reference" "R5"
-			(at 260.35 30.48 90)
+		(property "Reference" "SW1"
+			(at 100.33 27.9399 90)
 			(effects
 				(font
-					(size 1.016 1.016)
+					(size 1.27 1.27)
 				)
+				(justify right)
 			)
 		)
-		(property "Value" "1.5k"
-			(at 260.35 33.02 90)
+		(property "Value" "PWR SWITCH"
+			(at 100.33 30.4799 90)
 			(effects
 				(font
 					(size 1.27 1.27)
 				)
+				(justify right)
 			)
 		)
-		(property "Footprint" "Resistor_SMD:R_0603_1608Metric_Pad0.98x0.95mm_HandSolder"
-			(at 260.35 35.56 0)
+		(property "Footprint" "Connector_PinSocket_2.54mm:PinSocket_1x02_P2.54mm_Vertical"
+			(at 99.06 29.21 0)
 			(effects
 				(font
@@
 		)
 		(property "Datasheet" "~"
-			(at 260.35 35.56 0)
+			(at 99.06 29.21 0)
 			(effects
 				(font
@@
 			)
 		)
-		(property "Description" "Resistor, small symbol"
-			(at 260.35 35.56 0)
+		(property "Description" "Single Pole Single Throw (SPST) switch, separate symbol"
+			(at 99.06 29.21 0)
 			(effects
 				(font
@@
 			)
 		)
-		(pin "2"
-		)
 		(pin "1"
 		)
+		(pin "3"
+		)
+		(pin "4"
+		)
+		(pin "2"
+		)
 		(instances
-			(project "pcb"
+			(project ""
 				(path "/a02550bc-85b4-480d-868d-ccdfd0f6046d"
-					(reference "R5")
+					(reference "SW1")
 					(unit 1)
 				)
@@
 	)
 	(symbol
-		(lib_id "power:+3.3V")
-		(at 99.06 34.29 0)
+		(lib_id "Device:R_Small")
+		(at 260.35 35.56 90)
 		(unit 1)
 		(exclude_from_sim no)
@@
 		(dnp no)
 		(fields_autoplaced yes)
-		(property "Reference" "#PWR04"
-			(at 99.06 38.1 0)
+		(property "Reference" "R5"
+			(at 260.35 30.48 90)
 			(effects
 				(font
-					(size 1.27 1.27)
+					(size 1.016 1.016)
 				)
-				(hide yes)
 			)
 		)
-		(property "Value" "+3.3V"
-			(at 101.6 33.0199 0)
+		(property "Value" "1.5k"
+			(at 260.35 33.02 90)
 			(effects
 				(font
 					(size 1.27 1.27)
 				)
-				(justify left)
 			)
 		)
-		(property "Footprint" ""
-			(at 99.06 34.29 0)
+		(property "Footprint" "Resistor_SMD:R_0603_1608Metric_Pad0.98x0.95mm_HandSolder"
+			(at 260.35 35.56 0)
 			(effects
 				(font
@@
 			)
 		)
-		(property "Datasheet" ""
-			(at 99.06 34.29 0)
+		(property "Datasheet" "~"
+			(at 260.35 35.56 0)
 			(effects
 				(font
@@
 			)
 		)
-		(property "Description" "Power symbol creates a global label with name \"+3.3V\""
-			(at 99.06 34.29 0)
+		(property "Description" "Resistor, small symbol"
+			(at 260.35 35.56 0)
 			(effects
 				(font
@@
 			)
 		)
+		(pin "2"
+		)
 		(pin "1"
 		)
 		(instances
-			(project ""
+			(project "pcb"
 				(path "/a02550bc-85b4-480d-868d-ccdfd0f6046d"
-					(reference "#PWR04")
+					(reference "R5")
 					(unit 1)
 				)
@@
 					(unit 1)
 				)
+			)
+		)
+	)
+	(symbol
+		(lib_id "power:+3.3V")
+		(at 99.06 24.13 0)
+		(unit 1)
+		(exclude_from_sim no)
+		(in_bom yes)
+		(on_board yes)
+		(dnp no)
+		(fields_autoplaced yes)
+		(property "Reference" "#PWR04"
+			(at 99.06 27.94 0)
+			(effects
+				(font
+					(size 1.27 1.27)
+				)
+				(hide yes)
+			)
+		)
+		(property "Value" "+3.3V"
+			(at 101.6 22.8599 0)
+			(effects
+				(font
+					(size 1.27 1.27)
+				)
+				(justify left)
+			)
+		)
+		(property "Footprint" ""
+			(at 99.06 24.13 0)
+			(effects
+				(font
+					(size 1.27 1.27)
+				)
+				(hide yes)
+			)
+		)
+		(property "Datasheet" ""
+			(at 99.06 24.13 0)
+			(effects
+				(font
+					(size 1.27 1.27)
+				)
+				(hide yes)
+			)
+		)
+		(property "Description" "Power symbol creates a global label with name \"+3.3V\""
+			(at 99.06 24.13 0)
+			(effects
+				(font
+					(size 1.27 1.27)
+				)
+				(hide yes)
+			)
+		)
+		(pin "1"
+		)
+		(instances
+			(project "pcb"
+				(path "/a02550bc-85b4-480d-868d-ccdfd0f6046d"
+					(reference "#PWR04")
+					(unit 1)
+				)

Commit message: finish pcb
Parts:
- J1: footprint Connector_USB:USB_C_Receptacle_Amphenol_12401548E4-2A -> Connector_USB:USB_C_Receptacle_GCT_USB4125-xx-x-0190_6P_TopMnt_Horizontal
Changed lines of the file:
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@@
 			)
 		)
-		(property "Footprint" "Connector_USB:USB_C_Receptacle_Amphenol_12401548E4-2A"
+		(property "Footprint" "Connector_USB:USB_C_Receptacle_GCT_USB4125-xx-x-0190_6P_TopMnt_Horizontal"
 			(at 60.96 109.22 0)
 			(effects

Commit message: move capacitors closer
Parts:
- removed C8: 6.8pF, Capacitor_SMD:C_0603_1608Metric_Pad1.08x0.95mm_HandSolder, symbol Device:C_Small
Connections:
- net at C2.1, L1.2, R1.1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: now also R1.2, R2.1, U1.5 (FB)
Changed lines of the file:
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@@
 	(wire
 		(pts
-			(xy 99.06 34.29) (xy 99.06 36.83)
-		)
-		(stroke
-			(width 0)
-			(type default)
-		)
-	)
-	(wire
-		(pts
 			(xy 129.54 115.57) (xy 133.35 115.57)
 		)
@@
 	(wire
 		(pts
-			(xy 99.06 41.91) (xy 99.06 45.72)
+			(xy 99.06 34.29) (xy 99.06 45.72)
 		)
 		(stroke
@@
 					(unit 1)
 				)
-			)
-		)
-	)
-	(symbol
-		(lib_id "Device:C_Small")
-		(at 99.06 39.37 0)
-		(unit 1)
-		(exclude_from_sim no)
-		(in_bom yes)
-		(on_board yes)
-		(dnp no)
-		(fields_autoplaced yes)
-		(property "Reference" "C8"
-			(at 101.6 38.1062 0)
-			(effects
-				(font
-					(size 1.27 1.27)
-				)
-				(justify left)
-			)
-		)
-		(property "Value" "6.8pF"
-			(at 101.6 40.6462 0)
-			(effects
-				(font
-					(size 1.27 1.27)
-				)
-				(justify left)
-			)
-		)
-		(property "Footprint" "Capacitor_SMD:C_0603_1608Metric_Pad1.08x0.95mm_HandSolder"
-			(at 99.06 39.37 0)
-			(effects
-				(font
-					(size 1.27 1.27)
-				)
-				(hide yes)
-			)
-		)
-		(property "Datasheet" "~"
-			(at 99.06 39.37 0)
-			(effects
-				(font
-					(size 1.27 1.27)
-				)
-				(hide yes)
-			)
-		)
-		(property "Description" "Unpolarized capacitor, small symbol"
-			(at 99.06 39.37 0)
-			(effects
-				(font
-					(size 1.27 1.27)
-				)
-				(hide yes)
-			)
-		)
-		(pin "2"
-		)
-		(pin "1"
-		)
-		(instances
-			(project "pcb"
-				(path "/a02550bc-85b4-480d-868d-ccdfd0f6046d"
-					(reference "C8")
-					(unit 1)
-				)

Commit message: switch to grouped headers
Parts:
- removed J10: SWDIO, Connector_PinSocket_2.54mm:PinSocket_1x01_P2.54mm_Vertical, symbol Connector:Conn_01x01_Socket
- removed J11: SWCLK, Connector_PinSocket_2.54mm:PinSocket_1x01_P2.54mm_Vertical, symbol Connector:Conn_01x01_Socket
- removed J12: USART1 TX, Connector_PinSocket_2.54mm:PinSocket_1x01_P2.54mm_Vertical, symbol Connector:Conn_01x01_Socket
- removed J13: USART1 RX, Connector_PinSocket_2.54mm:PinSocket_1x01_P2.54mm_Vertical, symbol Connector:Conn_01x01_Socket
- removed J14, J16, J8: GND, Connector_PinSocket_2.54mm:PinSocket_1x01_P2.54mm_Vertical, symbol Connector:Conn_01x01_Socket
- removed J15, J6: 3.3v, Connector_PinSocket_2.54mm:PinSocket_1x01_P2.54mm_Vertical, symbol Connector:Conn_01x01_Socket
- removed J17: NRST, Connector_PinSocket_2.54mm:PinSocket_1x01_P2.54mm_Vertical, symbol Connector:Conn_01x01_Socket
- removed J2: +3.3V, Connector_PinSocket_2.54mm:PinSocket_1x01_P2.54mm_Vertical, symbol Connector:Conn_01x01_Socket
- removed J4: LCD RS, Connector_PinSocket_2.54mm:PinSocket_1x01_P2.54mm_Vertical, symbol Connector:Conn_01x01_Socket
- removed J5: LCD E, Connector_PinSocket_2.54mm:PinSocket_1x01_P2.54mm_Vertical, symbol Connector:Conn_01x01_Socket
- removed J7: ADC2, Connector_PinSocket_2.54mm:PinSocket_1x01_P2.54mm_Vertical, symbol Connector:Conn_01x01_Socket
- added J4: LCD CTRL, Connector_PinHeader_2.54mm:PinHeader_1x04_P2.54mm_Vertical, symbol Connector:Conn_01x04_Socket
- added J5: M SEN, Connector_PinHeader_2.54mm:PinHeader_1x03_P2.54mm_Vertical, symbol Connector:Conn_01x03_Socket
- added J6: HC-05, Connector_PinHeader_2.54mm:PinHeader_1x04_P2.54mm_Vertical, symbol Connector:Conn_01x04_Socket
- added J7: DEBUG, Connector_PinHeader_2.54mm:PinHeader_1x03_P2.54mm_Vertical, symbol Connector:Conn_01x03_Socket
Connections:
- net +3.3V: now also J4.3 (Pin_3), J5.2 (Pin_2), J6.3 (Pin_3)
- net GND: now also J4.4 (Pin_4), J5.3 (Pin_3), J6.4 (Pin_4)
- net NRST: now also J7.3 (Pin_3)
- net PA1 renamed ADC1
- net PA10 renamed USART1 RX
- net USART1 RX: now also J6.2 (Pin_2)
- net PA13 renamed SWDIO
- net SWDIO: now also J7.1 (Pin_1)
- net PA14 renamed SWCLK
- net SWCLK: now also J7.2 (Pin_2)
- net PA4 renamed ADC2
- net ADC2: now also J5.1 (Pin_1)
- net PA5 renamed SYS LED
- net PA9 renamed USART1 TX
- net USART1 TX: now also J6.1 (Pin_1)
- net PB10 renamed USART3 TX
- net PB13 renamed LCD RS
- net LCD RS: now also J4.1 (Pin_1)
- net PB15 renamed LCD E
- net LCD E: now also J4.2 (Pin_2)
- net PB8 renamed LCD D3
- net PC10 renamed LCD D5
- net PC11 renamed LCD D6
- net PC12 renamed LCD D7
- net PC6 renamed LCD D4
- net PC8 renamed LCD D2
- net PC9 renamed LCD D1
- net PD2 renamed LCD D8
- no-connect marks 38 -> 39
Other:
- moved on the sheet: J9

Commit message: redesign charging circuit
Connections:
- net +3.3V: now also C2.1, L1.2, R1.1, R1.2, R2.1, SW1.1 (A), U1.5 (FB)
Other:
- moved on the sheet: SW1A
Changed lines of the file:
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@@
 	)
 	(junction
-		(at 99.06 34.29)
-		(diameter 0)
-		(color 0 0 0 0)
-	)
-	(junction
 		(at 137.16 33.02)
 		(diameter 0)
@@
 	)
 	(junction
+		(at 99.06 34.29)
+		(diameter 0)
+		(color 0 0 0 0)
+	)
+	(junction
 		(at 148.59 154.94)
 		(diameter 0)
@@
 	(wire
 		(pts
+			(xy 99.06 31.75) (xy 99.06 34.29)
+		)
+		(stroke
+			(width 0)
+			(type default)
+		)
+	)
+	(wire
+		(pts
 			(xy 214.63 59.69) (xy 214.63 63.5)
 		)
@@
 	(wire
 		(pts
+			(xy 114.3 38.1) (xy 114.3 36.83)
+		)
+		(stroke
+			(width 0)
+			(type default)
+		)
+	)
+	(wire
+		(pts
 			(xy 182.88 105.41) (xy 173.99 105.41)
 		)
@@
 	(symbol
 		(lib_id "Switch:SW_DPST_x2")
-		(at 99.06 29.21 90)
+		(at 114.3 31.75 90)
 		(unit 1)
 		(exclude_from_sim no)
@@
 		(on_board yes)
 		(dnp no)
-		(fields_autoplaced yes)
 		(property "Reference" "SW1"
-			(at 100.33 27.9399 90)
+			(at 115.57 30.4799 90)
 			(effects
 				(font
@@
 		)
 		(property "Value" "PWR SWITCH"
-			(at 100.33 30.4799 90)
+			(at 115.57 33.0199 90)
 			(effects
 				(font
@@
 		)
 		(property "Footprint" "Connector_PinSocket_2.54mm:PinSocket_1x02_P2.54mm_Vertical"
-			(at 99.06 29.21 0)
+			(at 114.3 31.75 0)
 			(effects
 				(font
@@
 		)
 		(property "Datasheet" "~"
-			(at 99.06 29.21 0)
+			(at 114.3 31.75 0)
 			(effects
 				(font
@@
 		)
 		(property "Description" "Single Pole Single Throw (SPST) switch, separate symbol"
-			(at 99.06 29.21 0)
+			(at 114.3 31.75 0)
 			(effects
 				(font
@@
 	(symbol
 		(lib_id "power:+3.3V")
-		(at 99.06 24.13 0)
+		(at 114.3 26.67 0)
 		(unit 1)
 		(exclude_from_sim no)
@@
 		(fields_autoplaced yes)
 		(property "Reference" "#PWR04"
-			(at 99.06 27.94 0)
+			(at 114.3 30.48 0)
 			(effects
 				(font
@@
 		)
 		(property "Value" "+3.3V"
-			(at 101.6 22.8599 0)
+			(at 116.84 25.3999 0)
 			(effects
 				(font
@@
 		)
 		(property "Footprint" ""
-			(at 99.06 24.13 0)
+			(at 114.3 26.67 0)
 			(effects
 				(font
@@
 		)
 		(property "Datasheet" ""
-			(at 99.06 24.13 0)
+			(at 114.3 26.67 0)
 			(effects
 				(font
@@
 		)
 		(property "Description" "Power symbol creates a global label with name \"+3.3V\""
-			(at 99.06 24.13 0)
+			(at 114.3 26.67 0)
 			(effects
 				(font
@@
 	)
 	(symbol
+		(lib_id "power:+3.3V")
+		(at 99.06 31.75 0)
+		(unit 1)
+		(exclude_from_sim no)
+		(in_bom yes)
+		(on_board yes)
+		(dnp no)
+		(property "Reference" "#PWR028"
+			(at 99.06 35.56 0)
+			(effects
+				(font
+					(size 1.27 1.27)
+				)
+				(hide yes)
+			)
+		)
+		(property "Value" "+3.3V"
+			(at 97.79 27.178 0)
+			(effects
+				(font
+					(size 1.27 1.27)
+				)
+				(justify left)
+			)
+		)
+		(property "Footprint" ""
+			(at 99.06 31.75 0)
+			(effects
+				(font
+					(size 1.27 1.27)
+				)
+				(hide yes)
+			)
+		)
+		(property "Datasheet" ""
+			(at 99.06 31.75 0)
+			(effects
+				(font
+					(size 1.27 1.27)
+				)
+				(hide yes)
+			)
+		)
+		(property "Description" "Power symbol creates a global label with name \"+3.3V\""
+			(at 99.06 31.75 0)
+			(effects
+				(font
+					(size 1.27 1.27)
+				)
+				(hide yes)
+			)
+		)
+		(pin "1"
+		)
+		(instances
+			(project "pcb"
+				(path "/a02550bc-85b4-480d-868d-ccdfd0f6046d"
+					(reference "#PWR028")
+					(unit 1)
+				)
+			)
+		)
+	)
+	(symbol
 		(lib_id "Device:C_Small")
 		(at 207.01 30.48 0)
@@
 					(unit 1)
 				)
+			)
+		)
+	)
+	(symbol
+		(lib_id "power:+3.3V")
+		(at 114.3 38.1 180)
+		(unit 1)
+		(exclude_from_sim no)
+		(in_bom yes)
+		(on_board yes)
+		(dnp no)
+		(fields_autoplaced yes)
+		(property "Reference" "#PWR011"
+			(at 114.3 34.29 0)
+			(effects
+				(font
+					(size 1.27 1.27)
+				)
+				(hide yes)
+			)
+		)
+		(property "Value" "+3.3V"
+			(at 114.3 43.18 0)
+			(effects
+				(font
+					(size 1.27 1.27)
+				)
+			)
+		)
+		(property "Footprint" ""
+			(at 114.3 38.1 0)
+			(effects
+				(font
+					(size 1.27 1.27)
+				)
+				(hide yes)
+			)
+		)
+		(property "Datasheet" ""
+			(at 114.3 38.1 0)
+			(effects
+				(font
+					(size 1.27 1.27)
+				)
+				(hide yes)
+			)
+		)
+		(property "Description" "Power symbol creates a global label with name \"+3.3V\""
+			(at 114.3 38.1 0)
+			(effects
+				(font
+					(size 1.27 1.27)
+				)
+				(hide yes)
+			)
+		)
+		(pin "1"
+		)
+		(instances
+			(project ""
+				(path "/a02550bc-85b4-480d-868d-ccdfd0f6046d"
+					(reference "#PWR011")
+					(unit 1)
+				)

Commit message: fix errors and add labels
Parts:
- R7: value 82k -> 200k
Changed lines of the file:
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@@
 			)
 		)
-		(property "Value" "82k"
+		(property "Value" "200k"
 			(at 217.17 67.3099 0)
 			(effects
