File: pcb/pcb.kicad_sch (KiCad schematic)
At the start: 35 parts, among them J1 USB_C_Receptacle_USB2.0_14P, J3 LCD Data, J4 LCD CTRL, J5 M SEN, J6 HC-05, J7 DEBUG, J9 USART3 TX, SW1 PWR SWITCH, U1 TLV62569DBV, U2 STM32F446RETx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

Commit message: add vcap capacitor and widen traces
Parts:
- added C8: 4.7uF, Capacitor_SMD:C_0603_1608Metric_Pad1.08x0.95mm_HandSolder, symbol Device:C_Small
Connections:
- net +3.3V: no longer U2.30 (VCAP_1)
- net GND: now also C8.2
- new net: C8.1, U2.30 (VCAP_1)
Changed lines of the file:
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@@
 	(wire
 		(pts
+			(xy 180.34 77.47) (xy 181.61 77.47)
+		)
+		(stroke
+			(width 0)
+			(type default)
+		)
+	)
+	(wire
+		(pts
 			(xy 133.35 69.85) (xy 127 69.85)
 		)
@@
 	(wire
 		(pts
-			(xy 179.07 77.47) (xy 173.99 77.47)
+			(xy 175.26 77.47) (xy 173.99 77.47)
 		)
 		(stroke
@@
 	)
 	(symbol
-		(lib_id "power:+3.3V")
-		(at 269.24 24.13 0)
+		(lib_id "Device:C_Small")
+		(at 177.8 77.47 90)
 		(unit 1)
 		(exclude_from_sim no)
@@
 		(dnp no)
 		(fields_autoplaced yes)
-		(property "Reference" "#PWR010"
-			(at 269.24 27.94 0)
+		(property "Reference" "C8"
+			(at 176.5362 74.93 0)
 			(effects
 				(font
 					(size 1.27 1.27)
 				)
-				(hide yes)
+				(justify left)
 			)
 		)
-		(property "Value" "+3.3V"
-			(at 271.78 22.8599 0)
+		(property "Value" "4.7uF"
+			(at 179.0762 74.93 0)
 			(effects
 				(font
@@
 			)
 		)
-		(property "Footprint" ""
-			(at 269.24 24.13 0)
+		(property "Footprint" "Capacitor_SMD:C_0603_1608Metric_Pad1.08x0.95mm_HandSolder"
+			(at 177.8 77.47 0)
 			(effects
 				(font
@@
 			)
 		)
-		(property "Datasheet" ""
-			(at 269.24 24.13 0)
+		(property "Datasheet" "~"
+			(at 177.8 77.47 0)
 			(effects
 				(font
@@
 			)
 		)
-		(property "Description" "Power symbol creates a global label with name \"+3.3V\""
-			(at 269.24 24.13 0)
+		(property "Description" "Unpolarized capacitor, small symbol"
+			(at 177.8 77.47 0)
 			(effects
 				(font
@@
 			)
 		)
+		(pin "2"
+		)
 		(pin "1"
 		)
 		(instances
-			(project ""
+			(project "pcb"
 				(path "/a02550bc-85b4-480d-868d-ccdfd0f6046d"
-					(reference "#PWR010")
+					(reference "C8")
 					(unit 1)
 				)
@@
 	)
 	(symbol
-		(lib_id "power:+5V")
-		(at 78.74 93.98 0)
+		(lib_id "power:+3.3V")
+		(at 269.24 24.13 0)
 		(unit 1)
 		(exclude_from_sim no)
@@
 		(dnp no)
 		(fields_autoplaced yes)
-		(property "Reference" "#PWR026"
-			(at 78.74 97.79 0)
+		(property "Reference" "#PWR010"
+			(at 269.24 27.94 0)
 			(effects
 				(font
@@
 			)
 		)
-		(property "Value" "+5V"
-			(at 78.74 88.9 0)
+		(property "Value" "+3.3V"
+			(at 271.78 22.8599 0)
 			(effects
 				(font
 					(size 1.27 1.27)
 				)
+				(justify left)
 			)
 		)
 		(property "Footprint" ""
-			(at 78.74 93.98 0)
+			(at 269.24 24.13 0)
 			(effects
 				(font
@@
 		)
 		(property "Datasheet" ""
-			(at 78.74 93.98 0)
+			(at 269.24 24.13 0)
 			(effects
 				(font
@@
 			)
 		)
-		(property "Description" "Power symbol creates a global label with name \"+5V\""
-			(at 78.74 93.98 0)
+		(property "Description" "Power symbol creates a global label with name \"+3.3V\""
+			(at 269.24 24.13 0)
 			(effects
 				(font
@@
 			(project ""
 				(path "/a02550bc-85b4-480d-868d-ccdfd0f6046d"
-					(reference "#PWR026")
+					(reference "#PWR010")
 					(unit 1)
 				)
@@
 	)
 	(symbol
-		(lib_id "power:GND")
-		(at 251.46 81.28 270)
+		(lib_id "power:+5V")
+		(at 78.74 93.98 0)
 		(unit 1)
 		(exclude_from_sim no)
@@
 		(on_board yes)
 		(dnp no)
-		(property "Reference" "#PWR07"
-			(at 245.11 81.28 0)
+		(fields_autoplaced yes)
+		(property "Reference" "#PWR026"
+			(at 78.74 97.79 0)
 			(effects
 				(font
@@
 			)
 		)
-		(property "Value" "GND"
-			(at 245.11 81.788 0)
+		(property "Value" "+5V"
+			(at 78.74 88.9 0)
 			(effects
 				(font
@@
 		)
 		(property "Footprint" ""
-			(at 251.46 81.28 0)
+			(at 78.74 93.98 0)
 			(effects
 				(font
@@
 		)
 		(property "Datasheet" ""
-			(at 251.46 81.28 0)
+			(at 78.74 93.98 0)
 			(effects
 				(font
@@
 			)
 		)
-		(property "Description" "Power symbol creates a global label with name \"GND\" , ground"
-			(at 251.46 81.28 0)
+		(property "Description" "Power symbol creates a global label with name \"+5V\""
+			(at 78.74 93.98 0)
 			(effects
 				(font
@@
 		)
 		(instances
-			(project "pcb"
+			(project ""
 				(path "/a02550bc-85b4-480d-868d-ccdfd0f6046d"
-					(reference "#PWR07")
+					(reference "#PWR026")
 					(unit 1)
 				)
@@
 	)
 	(symbol
-		(lib_id "power:+3.3V")
-		(at 151.13 160.02 180)
+		(lib_id "power:GND")
+		(at 251.46 81.28 270)
 		(unit 1)
 		(exclude_from_sim no)
@@
 		(on_board yes)
 		(dnp no)
-		(fields_autoplaced yes)
-		(property "Reference" "#PWR06"
-			(at 151.13 156.21 0)
+		(property "Reference" "#PWR07"
+			(at 245.11 81.28 0)
 			(effects
 				(font
@@
 			)
 		)
-		(property "Value" "+3.3V"
-			(at 148.59 161.2901 0)
+		(property "Value" "GND"
+			(at 245.11 81.788 0)
 			(effects
 				(font
 					(size 1.27 1.27)
 				)
-				(justify left)
 			)
 		)
 		(property "Footprint" ""
-			(at 151.13 160.02 0)
+			(at 251.46 81.28 0)
 			(effects
 				(font
@@
 		)
 		(property "Datasheet" ""
-			(at 151.13 160.02 0)
+			(at 251.46 81.28 0)
 			(effects
 				(font
@@
 			)
 		)
-		(property "Description" "Power symbol creates a global label with name \"+3.3V\""
-			(at 151.13 160.02 0)
+		(property "Description" "Power symbol creates a global label with name \"GND\" , ground"
+			(at 251.46 81.28 0)
 			(effects
 				(font
@@
 			(project "pcb"
 				(path "/a02550bc-85b4-480d-868d-ccdfd0f6046d"
-					(reference "#PWR06")
+					(reference "#PWR07")
 					(unit 1)
 				)
@@
 	(symbol
 		(lib_id "power:+3.3V")
-		(at 179.07 77.47 270)
+		(at 151.13 160.02 180)
 		(unit 1)
 		(exclude_from_sim no)
@@
 		(dnp no)
 		(fields_autoplaced yes)
-		(property "Reference" "#PWR022"
-			(at 175.26 77.47 0)
+		(property "Reference" "#PWR06"
+			(at 151.13 156.21 0)
 			(effects
 				(font
@@
 		)
 		(property "Value" "+3.3V"
-			(at 180.3401 80.01 0)
+			(at 148.59 161.2901 0)
 			(effects
 				(font
@@
 		)
 		(property "Footprint" ""
-			(at 179.07 77.47 0)
+			(at 151.13 160.02 0)
 			(effects
 				(font
@@
 		)
 		(property "Datasheet" ""
-			(at 179.07 77.47 0)
+			(at 151.13 160.02 0)
 			(effects
 				(font
@@
 		)
 		(property "Description" "Power symbol creates a global label with name \"+3.3V\""
-			(at 179.07 77.47 0)
+			(at 151.13 160.02 0)
 			(effects
 				(font
@@
 			(project "pcb"
 				(path "/a02550bc-85b4-480d-868d-ccdfd0f6046d"
-					(reference "#PWR022")
+					(reference "#PWR06")
 					(unit 1)
 				)
@@
 					(unit 1)
 				)
+			)
+		)
+	)
+	(symbol
+		(lib_id "power:GND")
+		(at 181.61 77.47 90)
+		(unit 1)
+		(exclude_from_sim no)
+		(in_bom yes)
+		(on_board yes)
+		(dnp no)
+		(fields_autoplaced yes)
+		(property "Reference" "#PWR022"
+			(at 187.96 77.47 0)
+			(effects
+				(font
+					(size 1.27 1.27)
+				)
+				(hide yes)
+			)
+		)
+		(property "Value" "GND"
+			(at 186.69 77.47 0)
+			(effects
+				(font
+					(size 1.27 1.27)
+				)
+			)
+		)
+		(property "Footprint" ""
+			(at 181.61 77.47 0)
+			(effects
+				(font
+					(size 1.27 1.27)
+				)
+				(hide yes)
+			)
+		)
+		(property "Datasheet" ""
+			(at 181.61 77.47 0)
+			(effects
+				(font
+					(size 1.27 1.27)
+				)
+				(hide yes)
+			)
+		)
+		(property "Description" "Power symbol creates a global label with name \"GND\" , ground"
+			(at 181.61 77.47 0)
+			(effects
+				(font
+					(size 1.27 1.27)
+				)
+				(hide yes)
+			)
+		)
+		(pin "1"
+		)
+		(instances
+			(project "pcb"
+				(path "/a02550bc-85b4-480d-868d-ccdfd0f6046d"
+					(reference "#PWR022")
+					(unit 1)
+				)

Commit message: change design to use 0402 for buck converter
Parts:
- R1: value 900k -> 450k; footprint Resistor_SMD:R_0603_1608Metric_Pad0.98x0.95mm_HandSolder -> Resistor_SMD:R_0402_1005Metric_Pad0.72x0.64mm_HandSolder
- R2: value 200k -> 100k; footprint Resistor_SMD:R_0603_1608Metric_Pad0.98x0.95mm_HandSolder -> Resistor_SMD:R_0402_1005Metric_Pad0.72x0.64mm_HandSolder
Other:
- note added: "DEBUG"
- note added: "MOISTURE"
- note removed: "Debug"
- note removed: "Moisture Sensor"
Changed lines of the file:
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@@
 		)
 	)
-	(text "Moisture Sensor"
+	(text "MOISTURE"
 		(exclude_from_sim no)
 		(at 258.064 103.124 0)
@@
 		)
 	)
-	(text "Debug"
+	(text "DEBUG"
 		(exclude_from_sim no)
 		(at 213.36 109.474 0)
@@
 			)
 		)
-		(property "Value" "900k"
+		(property "Value" "450k"
 			(at 88.9 41.9099 0)
 			(effects
@@
 			)
 		)
-		(property "Footprint" "Resistor_SMD:R_0603_1608Metric_Pad0.98x0.95mm_HandSolder"
+		(property "Footprint" "Resistor_SMD:R_0402_1005Metric_Pad0.72x0.64mm_HandSolder"
 			(at 86.36 40.64 0)
 			(effects
@@
 			)
 		)
-		(property "Value" "200k"
+		(property "Value" "100k"
 			(at 88.9 52.0699 0)
 			(effects
@@
 			)
 		)
-		(property "Footprint" "Resistor_SMD:R_0603_1608Metric_Pad0.98x0.95mm_HandSolder"
+		(property "Footprint" "Resistor_SMD:R_0402_1005Metric_Pad0.72x0.64mm_HandSolder"
 			(at 86.36 50.8 0)
 			(effects
